File: Hardware/Carte course en cours.sch (EAGLE design)
At the start: 40 parts, among them J2 MICRO-SD_CARD_SOCKET, J3 AVR_SPI_PROG_3X2NS, U1 ATMEGA328P_TQFP, U2 MPU6050, U3 TXB0104, U4 V_REG_317DPACK, U5 V_REG_317SMD, U6 FT232RL, Y1 16MHz

Commit message: Add connectors
Parts:
- added J4: RC receiver, SparkFun-Connectors:CONN_02
- added J5: ESC, SparkFun-Connectors:CONN_02
- added J6: PWR IN, SparkFun-Connectors:CONN_02
Connections:
- removed net CD: J2.CD2, U1.PB1(OC1A)
- new net CARDDETECT: J2.CD2, U1.PD5(T1)
- new net ESC_OUT: J5.2, U1.PB1(OC1A)
- new net RC_IN: J4.2, U1.PD3(INT1)
- net CS: now also U1.PD4(XCK/T0); no longer U1.PB0(ICP)
- net GND: now also J4.1, J5.1, J6.1
- net VCC: now also J6.2
Other:
- note added: "CONNECTORS"
- note removed: "card detect"
Changed lines of the file:
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@@
 <part name="P+12" library="supply1" library_urn="urn:adsk.eagle:library:371" deviceset="+5V" device=""/>
 <part name="+3V7" library="supply1" library_urn="urn:adsk.eagle:library:371" deviceset="+3V3" device=""/>
+<part name="J4" library="SparkFun-Connectors" library_urn="urn:adsk.eagle:library:513" deviceset="CONN_02" device="" package3d_urn="urn:adsk.eagle:package:38039/1" value="RC receiver"/>
+<part name="J5" library="SparkFun-Connectors" library_urn="urn:adsk.eagle:library:513" deviceset="CONN_02" device="" package3d_urn="urn:adsk.eagle:package:38039/1" value="ESC"/>
+<part name="GND16" library="supply1" library_urn="urn:adsk.eagle:library:371" deviceset="GND" device=""/>
+<part name="GND17" library="supply1" library_urn="urn:adsk.eagle:library:371" deviceset="GND" device=""/>
+<part name="J6" library="SparkFun-Connectors" library_urn="urn:adsk.eagle:library:513" deviceset="CONN_02" device="" package3d_urn="urn:adsk.eagle:package:38039/1" value="PWR IN"/>
+<part name="GND18" library="supply1" library_urn="urn:adsk.eagle:library:371" deviceset="GND" device=""/>
+<part name="P+13" library="supply1" library_urn="urn:adsk.eagle:library:371" deviceset="VCC" device=""/>
 </parts>
 <sheets>
 <sheet>
 <plain>
-<text x="256.54" y="132.08" size="1.778" layer="91">card detect</text>
 <wire x1="272.796" y1="111.76" x2="167.64" y2="111.76" width="0.6096" layer="94" style="longdash"/>
 <wire x1="167.64" y1="111.76" x2="167.64" y2="104.14" width="0.6096" layer="94" style="longdash"/>
-<wire x1="167.64" y1="104.14" x2="167.64" y2="0.254" width="0.6096" layer="94" style="longdash"/>
+<wire x1="167.64" y1="104.14" x2="167.64" y2="71.12" width="0.6096" layer="94" style="longdash"/>
+<wire x1="167.64" y1="71.12" x2="167.64" y2="0.254" width="0.6096" layer="94" style="longdash"/>
 <wire x1="167.64" y1="111.76" x2="167.64" y2="178.816" width="0.6096" layer="94" style="longdash"/>
 <wire x1="0.254" y1="119.38" x2="88.9" y2="119.38" width="0.6096" layer="94" style="longdash"/>
 <wire x1="88.9" y1="119.38" x2="96.52" y2="119.38" width="0.6096" layer="94" style="longdash"/>
 <wire x1="96.52" y1="119.38" x2="96.52" y2="104.14" width="0.6096" layer="94" style="longdash"/>
-<wire x1="96.52" y1="104.14" x2="96.52" y2="0.254" width="0.6096" layer="94" style="longdash"/>
+<wire x1="96.52" y1="104.14" x2="96.52" y2="71.12" width="0.6096" layer="94" style="longdash"/>
+<wire x1="96.52" y1="71.12" x2="96.52" y2="0.254" width="0.6096" layer="94" style="longdash"/>
 <wire x1="167.64" y1="104.14" x2="96.52" y2="104.14" width="0.6096" layer="94" style="longdash"/>
 <text x="10.16" y="7.62" size="6.4516" layer="94" font="vector" ratio="12">MCU</text>
 <text x="210.82" y="116.84" size="6.4516" layer="94" font="vector" ratio="12">SD</text>
 <text x="248.92" y="96.52" size="6.4516" layer="94" font="vector" ratio="12">IMU</text>
-<text x="129.54" y="167.64" size="6.4516" layer="94" font="vector" ratio="12">FTDI</text>
+<text x="134.62" y="165.1" size="6.4516" layer="94" font="vector" ratio="12">FTDI</text>
 <text x="5.08" y="124.46" size="6.4516" layer="94" font="vector" ratio="12">PSU</text>
 <wire x1="88.9" y1="119.38" x2="88.9" y2="178.816" width="0.6096" layer="94" style="longdash"/>
 <text x="182.88" y="22.86" size="2.54" layer="94" font="vector" ratio="12">Released under the GNU General Public License v3.0</text>
+<wire x1="167.64" y1="71.12" x2="96.52" y2="71.12" width="0.6096" layer="94" style="longdash"/>
+<text x="109.22" y="73.66" size="6.4516" layer="94" font="vector" ratio="12">CONNECTORS</text>
 </plain>
 <instances>
@@
 <instance part="P+12" gate="1" x="266.7" y="147.32" rot="MR0"/>
 <instance part="+3V7" gate="G$1" x="259.08" y="175.26" rot="MR0"/>
+<instance part="J4" gate="G$1" x="137.16" y="91.44" rot="MR0"/>
+<instance part="J5" gate="G$1" x="162.56" y="91.44" rot="MR0"/>
+<instance part="GND16" gate="1" x="127" y="86.36"/>
+<instance part="GND17" gate="1" x="152.4" y="86.36"/>
+<instance part="J6" gate="G$1" x="114.3" y="91.44" rot="MR0"/>
+<instance part="GND18" gate="1" x="104.14" y="86.36"/>
+<instance part="P+13" gate="VCC" x="104.14" y="99.06"/>
 </instances>
 <busses>
@@
 <wire x1="12.7" y1="157.48" x2="12.7" y2="162.56" width="0.1524" layer="91"/>
 <junction x="12.7" y="162.56"/>
+</segment>
+<segment>
+<pinref part="P+13" gate="VCC" pin="VCC"/>
+<pinref part="J6" gate="G$1" pin="2"/>
+<wire x1="104.14" y1="96.52" x2="104.14" y2="93.98" width="0.1524" layer="91"/>
+<wire x1="104.14" y1="93.98" x2="106.68" y2="93.98" width="0.1524" layer="91"/>
 </segment>
 </net>
@@
 <pinref part="GND15" gate="1" pin="GND"/>
 </segment>
+<segment>
+<pinref part="J5" gate="G$1" pin="1"/>
+<pinref part="GND17" gate="1" pin="GND"/>
+<wire x1="154.94" y1="91.44" x2="152.4" y2="91.44" width="0.1524" layer="91"/>
+<wire x1="152.4" y1="91.44" x2="152.4" y2="88.9" width="0.1524" layer="91"/>
+</segment>
+<segment>
+<pinref part="J4" gate="G$1" pin="1"/>
+<pinref part="GND16" gate="1" pin="GND"/>
+<wire x1="129.54" y1="91.44" x2="127" y2="91.44" width="0.1524" layer="91"/>
+<wire x1="127" y1="91.44" x2="127" y2="88.9" width="0.1524" layer="91"/>
+</segment>
+<segment>
+<pinref part="J6" gate="G$1" pin="1"/>
+<pinref part="GND18" gate="1" pin="GND"/>
+<wire x1="106.68" y1="91.44" x2="104.14" y2="91.44" width="0.1524" layer="91"/>
+<wire x1="104.14" y1="91.44" x2="104.14" y2="88.9" width="0.1524" layer="91"/>
+</segment>
 </net>
 <net name="N$1" class="0">
@@
 <net name="CS" class="0">
 <segment>
-<pinref part="U1" gate="U$1" pin="PB0(ICP)"/>
-<wire x1="73.66" y1="45.72" x2="76.2" y2="45.72" width="0.1524" layer="91"/>
-<label x="76.2" y="45.72" size="1.778" layer="95"/>
-</segment>
-<segment>
 <pinref part="U3" gate="G$1" pin="A1"/>
 <wire x1="180.34" y1="147.32" x2="177.8" y2="147.32" width="0.1524" layer="91"/>
 <label x="177.8" y="147.32" size="1.778" layer="95" rot="MR0"/>
+</segment>
+<segment>
+<pinref part="U1" gate="U$1" pin="PD4(XCK/T0)"/>
+<wire x1="73.66" y1="58.42" x2="76.2" y2="58.42" width="0.1524" layer="91"/>
+<label x="76.2" y="58.42" size="1.778" layer="95" ratio="12"/>
 </segment>
 </net>
@@
 </segment>
 </net>
-<net name="CD" class="0">
+<net name="RC_IN" class="0">
+<segment>
+<pinref part="J4" gate="G$1" pin="2"/>
+<wire x1="129.54" y1="93.98" x2="127" y2="93.98" width="0.1524" layer="91"/>
+<label x="127" y="93.98" size="1.778" layer="95" ratio="12" rot="MR0"/>
+</segment>
+<segment>
+<pinref part="U1" gate="U$1" pin="PD3(INT1)"/>
+<wire x1="73.66" y1="60.96" x2="76.2" y2="60.96" width="0.1524" layer="91"/>
+<label x="76.2" y="60.96" size="1.778" layer="95" ratio="12"/>
+</segment>
+</net>
+<net name="ESC_OUT" class="0">
+<segment>
+<pinref part="J5" gate="G$1" pin="2"/>
+<wire x1="154.94" y1="93.98" x2="152.4" y2="93.98" width="0.1524" layer="91"/>
+<label x="152.4" y="93.98" size="1.778" layer="95" ratio="12" rot="MR0"/>
+</segment>
+<segment>
+<pinref part="U1" gate="U$1" pin="PB1(OC1A)"/>
+<wire x1="73.66" y1="43.18" x2="76.2" y2="43.18" width="0.1524" layer="91"/>
+<label x="76.2" y="43.18" size="1.778" layer="95"/>
+</segment>
+</net>
+<net name="CARDDETECT" class="0">
+<segment>
+<pinref part="U1" gate="U$1" pin="PD5(T1)"/>
+<wire x1="73.66" y1="55.88" x2="76.2" y2="55.88" width="0.1524" layer="91"/>
+<label x="76.2" y="55.88" size="1.778" layer="95" ratio="12"/>
+</segment>
 <segment>
 <pinref part="J2" gate="1" pin="CD2"/>
@@
 <label x="256.54" y="134.62" size="1.778" layer="95"/>
 </segment>
-<segment>
-<pinref part="U1" gate="U$1" pin="PB1(OC1A)"/>
-<wire x1="73.66" y1="43.18" x2="76.2" y2="43.18" width="0.1524" layer="91"/>
-<label x="76.2" y="43.18" size="1.778" layer="95"/>
-</segment>
-</net>
+</net>

Commit message: Add brd file
Parts:
- C1, C8: value 1u -> 4.7u
- C10, C9: value 22p -> 100n
- C12: value 4.7u -> 100n
- C2: value 4.7u -> 22p
- C3: value 100n -> 22p
- C4, C7: value 100n -> 1u
- J1: value (none) -> AVR_SPI_PROG_3X2NS; device SparkFun-Connectors:USB_MICRO-B_FEMALE-SMT -> SparkFun-Connectors:AVR_SPI_PROG_3X2NS
- J2: value MICRO-SD_CARD_SOCKET -> (none); device SparkFun-Connectors:MICRO-SD_CARD_SOCKET -> SparkFun-Connectors:USB_MICRO-B_FEMALE-SMT
- J3: value AVR_SPI_PROG_3X2NS -> PWR IN; device SparkFun-Connectors:AVR_SPI_PROG_3X2NS -> SparkFun-Connectors:CONN_02
- J6: value PWR IN -> MICRO-SD_CARD_SOCKET; device SparkFun-Connectors:CONN_02 -> SparkFun-Connectors:MICRO-SD_CARD_SOCKET
- R1: value 10k -> 3k
- R10: value 3k -> 100k
- R11: value 1k -> 100k
- R12, R13: value 330 -> 100k
- R2: value 4.7k -> 10k
- R3: value 4.7k -> 1k
- R4: value 100k -> 1.6k
- R5: value 100k -> 1k
- R6, R7: value 100k -> 330
- R8: value 1.6k -> 4.7k
- R9: value 1k -> 4.7k
- U1: value ATMEGA328P_TQFP -> V_REG_317DPACK; device SparkFun-IC-Microcontroller:ATMEGA328P_TQFP -> SparkFun-IC-Power:V_REG_317DPACK
- U2: value MPU6050 -> ATMEGA328P_TQFP; device invensense:MPU6050 -> SparkFun-IC-Microcontroller:ATMEGA328P_TQFP
- U3: value TXB0104 -> V_REG_317SMD; device SparkFun-IC-Comms:TXB0104PWR -> SparkFun-IC-Power:V_REG_317SMD
- U4: value V_REG_317DPACK -> FT232RL; device SparkFun-IC-Power:V_REG_317DPACK -> SparkFun-IC-Comms:FT232RL-BASICSSOP
- U5: value V_REG_317SMD -> TXB0104; device SparkFun-IC-Power:V_REG_317SMD -> SparkFun-IC-Comms:TXB0104PWR
- U6: value FT232RL -> MPU6050; device SparkFun-IC-Comms:FT232RL-BASICSSOP -> invensense:MPU6050
Connections:
- net +3V3: now also C11.1, C12.1, C7.1, J6.VCC, R10.2, R11.1, R13.1, R8.2, R9.2, U3.OUT, U5.VCCB, U6.VDD; no longer C5.1, C6.1, C8.1, J2.VCC, R2.2, R3.2, R4.2, R6.1, R9.1, U2.VDD, U3.VCCB, U5.OUT
- net +5V: now also C10.1, C4.1, C5.2, C6.2, C8.2, C9.2, J1.2, J2.VBUS, R12.1, R2.2, R3.1, U1.OUT, U2.AVCC, U2.VCC@4, U2.VCC@6, U3.IN, U4.VCC, U4.VCCIO, U5.VCCA; no longer C1.1, C11.2, C12.2, C3.2, C4.2, C7.1, J1.VBUS, J3.2, R1.2, R11.1, R7.1, U1.AVCC, U1.VCC@4, U1.VCC@6, U3.VCCA, U4.OUT, U5.IN, U6.VCC, U6.VCCIO
- net CARDDETECT: now also J6.CD2, U2.PD5(T1); no longer J2.CD2, U1.PD5(T1)
- net CS: now also U2.PD4(XCK/T0), U5.A1; no longer U1.PD4(XCK/T0), U3.A1
- net ESC_OUT: now also U2.PB1(OC1A); no longer U1.PB1(OC1A)
- net GND: now also C1.1, C11.2, C12.2, C2.2, C3.2, C4.2, C5.1, C6.1, C8.1, C9.1, J1.6, J3.1, J6.GND, J6.SHIELD@1, J6.SHIELD@3, R1.1, R4.1, U2.AGND, U2.GND@3, U2.GND@5, U4.AGND, U4.GND1, U4.GND2, U4.GND3, U4.TEST, U5.GND, U6.AD0, U6.CLKIN, U6.FSYNC, U6.GND; no longer C1.2, C11.1, C12.1, C2.1, C3.1, C4.1, C5.2, C6.2, C8.2, C9.2, J1.GND, J2.SHIELD@1, J2.SHIELD@3, J3.6, J6.1, R10.1, R8.1, U1.AGND, U1.GND@3, U1.GND@5, U2.AD0, U2.CLKIN, U2.FSYNC, U2.GND, U3.GND, U6.AGND, U6.GND1, U6.GND2, U6.GND3, U6.TEST
- net INT: now also U2.PD2(INT0), U6.INT; no longer U1.PD2(INT0), U2.INT
- net MISO: now also J1.1, U2.PB4(MISO), U5.A4; no longer J3.1, U1.PB4(MISO), U3.A4
- net MOSI: now also J1.4, U2.PB3(MOSI/OC2), U5.A2; no longer J3.4, U1.PB3(MOSI/OC2), U3.A2
- net N$1: now also R1.2, R3.2, U1.ADJ; no longer R10.2, R11.2, U4.ADJ
- net N$10: now also U6.CPOUT; no longer U2.CPOUT
- net N$11: now also J6.!CS, R10.1, U5.B1; no longer J2.!CS, R4.1, U3.B1
- net N$12: now also R6.1, U4.TXLED; no longer R12.1, U6.TXLED
- net N$13: now also R7.1, U4.RXLED; no longer R13.1, U6.RXLED
- net N$14: now also R6.2; no longer R12.2
- net N$15: now also R7.2; no longer R13.2
- net N$16: now also U6.REGOUT; no longer U2.REGOUT
- net N$17: now also J6.DI, U5.B2; no longer J2.DI, U3.B2
- net N$18: now also U6.VLOGIC; no longer U2.VLOGIC
- net N$19: now also J6.SCK, U5.B3; no longer J2.SCK, U3.B3
- net N$2: now also J2.D-, U4.USBDM; no longer J1.D-, U6.USBDM
- net N$20: now also J6.DO, U5.B4; no longer J2.DO, U3.B4
- net N$27: now also J6.RSV@1, R11.2; no longer J2.RSV@1, R5.2
- net N$28: now also J6.RSV@2, R13.2; no longer J2.RSV@2, R6.2
- net N$29: now also J6.CD1, R12.2; no longer J2.CD1, R7.2
- net N$3: now also R4.2, R5.2, U3.ADJ; no longer R8.2, R9.2, U5.ADJ
- net N$5: now also C2.1, U2.PB6(XTAL1/TOSC1); no longer C9.1, U1.PB6(XTAL1/TOSC1)
- net N$6: now also C3.1, U2.PB7(XTAL2/TOSC2); no longer C10.1, U1.PB7(XTAL2/TOSC2)
- net N$7: now also J2.D+, U4.USBDP; no longer J1.D+, U6.USBDP
- net RC_IN: now also U2.PD3(INT1); no longer U1.PD3(INT1)
- net RST: now also J1.5, R2.1, U2.PC6(/RESET); no longer J3.5, R1.1, U1.PC6(/RESET)
- net RXFTDI: now also U2.PD1(TXD), U4.RXD; no longer U1.PD1(TXD), U6.RXD
- net SCK: now also J1.3, U2.PB5(SCK), U5.A3; no longer J3.3, U1.PB5(SCK), U3.A3
- net SCL: now also R8.1, U2.PC5(ADC5/SCL), U6.SCL; no longer R3.1, U1.PC5(ADC5/SCL), U2.SCL
- net SDA: now also R9.1, U2.PC4(ADC4/SDA), U6.SDA; no longer R2.1, U1.PC4(ADC4/SDA), U2.SDA
- net TXFTDI: now also U2.PD0(RXD), U4.TXD; no longer U1.PD0(RXD), U6.TXD
- net VCC: now also C1.2, J3.2, U1.IN; no longer C2.2, J6.2, U4.IN
Other:
- moved on the sheet: C1, C10, C11, C12, C2, C3, C4, C5, C6, C7, C8, C9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

Commit message: Place components
Parts:
- removed C13: 100n, rcl:C-EUC0805
- removed C14: 2.2n, rcl:C-EUC0805
- removed C15: 10n, rcl:C-EUC0805
- removed R13: 100k, rcl:R-EU_R0805
- removed U5: TXB0104, SparkFun-IC-Comms:TXB0104PWR
- removed U6: MPU6050, invensense:MPU6050
- added J7: MICRO-SD_CARD_SOCKET, SparkFun-Connectors:MICRO-SD_CARD_SOCKET
- added J8: ESC, SparkFun-Connectors:CONN_02
- C1: value 4.7u -> 22p
- C11: value 100n -> 2.2n
- C12: value 100n -> 10n
- C3: value 22p -> 100n
- C4: value 1u -> 100n
- C6: value 100n -> 4.7u
- C8: value 4.7u -> 100n
- J1: value AVR_SPI_PROG_3X2NS -> (none); device SparkFun-Connectors:AVR_SPI_PROG_3X2NS -> SparkFun-Connectors:USB_MICRO-B_FEMALE-SMT
- J2: value (none) -> AVR_SPI_PROG_3X2NS; device SparkFun-Connectors:USB_MICRO-B_FEMALE-SMT -> SparkFun-Connectors:AVR_SPI_PROG_3X2NS
- J6: value MICRO-SD_CARD_SOCKET -> ESC; device SparkFun-Connectors:MICRO-SD_CARD_SOCKET -> SparkFun-Connectors:CONN_02
- R1: value 3k -> 10k
- R2: value 10k -> 1.6k
- R4: value 1.6k -> 330
- R5: value 1k -> 330
- R6, R7: value 330 -> 100k
- U1: value V_REG_317DPACK -> V_REG_317SMD; device SparkFun-IC-Power:V_REG_317DPACK -> SparkFun-IC-Power:V_REG_317SMD
- U3: value V_REG_317SMD -> FT232RL; device SparkFun-IC-Power:V_REG_317SMD -> SparkFun-IC-Comms:FT232RL-BASICSSOP
- U4: value FT232RL -> MPU6050; device SparkFun-IC-Comms:FT232RL-BASICSSOP -> invensense:MPU6050
Connections:
- removed net N$11: J6.!CS, R10.1, U5.B1
- removed net N$17: J6.DI, U5.B2
- removed net N$19: J6.SCK, U5.B3
- removed net N$20: J6.DO, U5.B4
- removed net N$3: R4.2, R5.2, U3.ADJ
- removed net RXFTDI: U2.PD1(TXD), U4.RXD
- removed net TXFTDI: U2.PD0(RXD), U4.TXD
- removed net VCC: C1.2, J3.2, U1.IN
- new net RX_AVR: R7.2, U2.PD0(RXD), U3.TXD
- new net RX_ESP: J5.2, R6.1
- new net TX_AVR: R6.2, U2.PD1(TXD), U3.RXD
- new net TX_ESP: J8.1, R7.1
- net +3V3: now also C3.2, C4.2, C5.2, C6.2, C8.1, C9.1, J2.2, J3.2, J7.VCC, J8.2, LED1.A, LED2.A, R1.2, R10.1, R12.1, R3.1, U1.OUT, U2.AVCC, U2.VCC@4, U2.VCC@6, U3.VCC, U3.VCCIO, U4.VDD; no longer C11.1, C12.1, J6.VCC, R10.2, R13.1, R5.1, U3.OUT, U5.VCCB, U6.VDD
- net +5V: now also J1.VBUS, U1.IN; no longer C10.1, C4.1, C5.2, C6.2, C8.2, C9.2, J1.2, J2.VBUS, LED1.A, LED2.A, R12.1, R2.2, R3.1, U1.OUT, U2.AVCC, U2.VCC@4, U2.VCC@6, U3.IN, U4.VCC, U4.VCCIO, U5.VCCA
- net CARDDETECT: now also J7.CD2; no longer J6.CD2
- net CS: now also J7.!CS; no longer U5.A1
- net ESC_OUT: now also J6.2; no longer J5.2
- net GND: now also C1.2, C3.1, C4.1, C8.2, C9.2, J1.GND, J2.6, J6.1, J7.GND, J7.SHIELD@1, J7.SHIELD@3, R2.1, U3.AGND, U3.GND1, U3.GND2, U3.GND3, U3.TEST, U4.AD0, U4.CLKIN, U4.FSYNC, U4.GND; no longer C1.1, C13.2, C14.2, C15.2, C3.2, C4.2, C8.1, C9.1, J1.6, J2.GND, J6.GND, J6.SHIELD@1, J6.SHIELD@3, R1.1, R4.1, U4.AGND, U4.GND1, U4.GND2, U4.GND3, U4.TEST, U5.GND, U6.AD0, U6.CLKIN, U6.FSYNC, U6.GND
- net INT: now also U4.INT; no longer U6.INT
- net MISO: now also J2.1, J7.DO; no longer J1.1, U5.A4
- net MOSI: now also J2.4, J7.DI; no longer J1.4, U5.A2
- net N$1: now also R2.2; no longer R1.2
- net N$10: now also C11.1, U4.CPOUT; no longer C14.1, U6.CPOUT
- net N$12: now also R4.1, U3.TXLED; no longer R6.1, U4.TXLED
- net N$13: now also R5.1, U3.RXLED; no longer R7.1, U4.RXLED
- net N$14: now also R4.2; no longer R6.2
- net N$15: now also R5.2; no longer R7.2
- net N$16: now also C10.1, U4.REGOUT; no longer C13.1, U6.REGOUT
- net N$18: now also C12.1, U4.VLOGIC; no longer C15.1, U6.VLOGIC
- net N$2: now also J1.D-, U3.USBDM; no longer J2.D-, U4.USBDM
- net N$27: now also J7.RSV@1, R10.2; no longer J6.RSV@1, R11.2
- net N$28: now also J7.RSV@2, R12.2; no longer J6.RSV@2, R13.2
- net N$29: now also J7.CD1, R11.2; no longer J6.CD1, R12.2
- net N$5: now also C1.1; no longer C2.1
- net N$6: now also C2.1; no longer C3.1
- net N$7: now also J1.D+, U3.USBDP; no longer J2.D+, U4.USBDP
- net RST: now also J2.5, R1.1; no longer J1.5, R2.1
- net SCK: now also J2.3, J7.SCK; no longer J1.3, U5.A3
- net SCL: now also U4.SCL; no longer U6.SCL
- net SDA: now also U4.SDA; no longer U6.SDA
Other:
- note removed: "PSU"
- moved on the sheet: C1, C10, C11, C12, C2, C3, C4, C5, C6, C7, C8, C9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

Commit message: Route
Parts:
- added J9: (no value), SparkFun-Connectors:CONN_04
Connections:
- net +5V: now also J9.4
- net GND: now also J9.1
- net N$2: now also J9.3
- net N$7: now also J9.2
Other:
- moved on the sheet: J1
Changed lines of the file:
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@@
 <setting verticaltext="up"/>
 </settings>
-<grid distance="0.1" unitdist="inch" unit="inch" style="lines" multiple="1" display="no" altdistance="0.01" altunitdist="inch" altunit="mil"/>
+<grid distance="0.1" unitdist="inch" unit="inch" style="lines" multiple="1" display="no" altdistance="0.01" altunitdist="inch" altunit="inch"/>
 <layers>
 <layer number="1" name="Top" color="4" fill="1" visible="no" active="no"/>
@@
 <part name="J5" library="SparkFun-Connectors" library_urn="urn:adsk.eagle:library:513" deviceset="CONN_02" device="" package3d_urn="urn:adsk.eagle:package:38039/1" value="ESC"/>
 <part name="J8" library="SparkFun-Connectors" library_urn="urn:adsk.eagle:library:513" deviceset="CONN_02" device="" package3d_urn="urn:adsk.eagle:package:38039/1" value="ESC"/>
+<part name="J9" library="SparkFun-Connectors" library_urn="urn:adsk.eagle:library:513" deviceset="CONN_04" device="" package3d_urn="urn:adsk.eagle:package:38085/1"/>
 </parts>
 <sheets>
@@
 <instance part="GND7" gate="1" x="83.82" y="106.68"/>
 <instance part="U3" gate="G$1" x="88.9" y="160.02"/>
-<instance part="J1" gate="G$1" x="10.16" y="162.56" rot="MR90"/>
+<instance part="J1" gate="G$1" x="10.16" y="170.18" rot="MR90"/>
 <instance part="GND1" gate="1" x="5.08" y="152.4"/>
 <instance part="C3" gate="G$1" x="63.5" y="154.94" rot="MR180"/>
@@
 <instance part="J5" gate="G$1" x="154.94" y="96.52" rot="MR0"/>
 <instance part="J8" gate="G$1" x="154.94" y="104.14" rot="MR0"/>
+<instance part="J9" gate="G$1" x="10.16" y="142.24" rot="MR90"/>
 </instances>
 <busses>
@@
 <pinref part="GND1" gate="1" pin="GND"/>
 <wire x1="5.08" y1="154.94" x2="5.08" y2="157.48" width="0.1524" layer="91"/>
+<pinref part="J9" gate="G$1" pin="1"/>
+<wire x1="5.08" y1="157.48" x2="5.08" y2="165.1" width="0.1524" layer="91"/>
+<wire x1="5.08" y1="157.48" x2="7.62" y2="157.48" width="0.1524" layer="91"/>
+<wire x1="7.62" y1="157.48" x2="7.62" y2="147.32" width="0.1524" layer="91"/>
+<junction x="5.08" y="157.48"/>
 </segment>
 <segment>
@@
 <segment>
 <pinref part="J1" gate="G$1" pin="VBUS"/>
-<wire x1="15.24" y1="157.48" x2="15.24" y2="154.94" width="0.1524" layer="91"/>
-<wire x1="15.24" y1="154.94" x2="25.4" y2="154.94" width="0.1524" layer="91"/>
-<wire x1="25.4" y1="154.94" x2="25.4" y2="170.18" width="0.1524" layer="91"/>
+<wire x1="15.24" y1="165.1" x2="15.24" y2="162.56" width="0.1524" layer="91"/>
+<wire x1="15.24" y1="162.56" x2="25.4" y2="162.56" width="0.1524" layer="91"/>
+<wire x1="25.4" y1="162.56" x2="25.4" y2="170.18" width="0.1524" layer="91"/>
 <pinref part="P+1" gate="1" pin="+5V"/>
 <pinref part="U1" gate="G$1" pin="IN"/>
@@
 <wire x1="27.94" y1="170.18" x2="25.4" y2="170.18" width="0.1524" layer="91"/>
 <junction x="25.4" y="170.18"/>
+<pinref part="J9" gate="G$1" pin="4"/>
+<wire x1="15.24" y1="162.56" x2="15.24" y2="147.32" width="0.1524" layer="91"/>
+<junction x="15.24" y="162.56"/>
 </segment>
 </net>
@@
 <segment>
 <pinref part="J1" gate="G$1" pin="D-"/>
-<wire x1="12.7" y1="157.48" x2="12.7" y2="142.24" width="0.1524" layer="91"/>
-<wire x1="12.7" y1="142.24" x2="55.88" y2="142.24" width="0.1524" layer="91"/>
+<wire x1="12.7" y1="165.1" x2="12.7" y2="154.94" width="0.1524" layer="91"/>
+<wire x1="12.7" y1="154.94" x2="25.4" y2="154.94" width="0.1524" layer="91"/>
+<wire x1="25.4" y1="154.94" x2="25.4" y2="142.24" width="0.1524" layer="91"/>
+<wire x1="25.4" y1="142.24" x2="55.88" y2="142.24" width="0.1524" layer="91"/>
 <wire x1="55.88" y1="142.24" x2="55.88" y2="172.72" width="0.1524" layer="91"/>
 <wire x1="55.88" y1="172.72" x2="73.66" y2="172.72" width="0.1524" layer="91"/>
 <pinref part="U3" gate="G$1" pin="USBDM"/>
+<pinref part="J9" gate="G$1" pin="3"/>
+<wire x1="12.7" y1="154.94" x2="12.7" y2="147.32" width="0.1524" layer="91"/>
+<junction x="12.7" y="154.94"/>
 </segment>
 </net>
@@
 <pinref part="J1" gate="G$1" pin="D+"/>
 <pinref part="U3" gate="G$1" pin="USBDP"/>
-<wire x1="10.16" y1="157.48" x2="10.16" y2="139.7" width="0.1524" layer="91"/>
-<wire x1="10.16" y1="139.7" x2="58.42" y2="139.7" width="0.1524" layer="91"/>
-<wire x1="58.42" y1="139.7" x2="58.42" y2="170.18" width="0.1524" layer="91"/>
+<wire x1="10.16" y1="165.1" x2="10.16" y2="152.4" width="0.1524" layer="91"/>
+<wire x1="10.16" y1="152.4" x2="22.86" y2="152.4" width="0.1524" layer="91"/>
+<wire x1="22.86" y1="152.4" x2="22.86" y2="139.7" width="0.1524" layer="91"/>
+<wire x1="22.86" y1="139.7" x2="58.42" y2="139.7" width="0.1524" layer="91"/>
+<wire x1="58.42" y1="139.7" x2="58.42" y2="142.24" width="0.1524" layer="91"/>
+<wire x1="58.42" y1="142.24" x2="58.42" y2="152.4" width="0.1524" layer="91"/>
+<wire x1="58.42" y1="152.4" x2="58.42" y2="170.18" width="0.1524" layer="91"/>
 <wire x1="58.42" y1="170.18" x2="73.66" y2="170.18" width="0.1524" layer="91"/>
-</segment>
-</net>
+<pinref part="J9" gate="G$1" pin="2"/>
+<wire x1="10.16" y1="152.4" x2="10.16" y2="147.32" width="0.1524" layer="91"/>
+<junction x="10.16" y="152.4"/>
+</segment>
+</net>
